File: 2056-LPC546xxJyyyBD208-breakout.sch (KiCad schematic (older format))
At the start: 105 parts, among them J1 0548190519, J10 Conn_01x03, J11 Conn_01x03, J12 Conn_01x03, J13 Conn_01x03, J14 Conn_01x03, J15 Conn_01x03, J16 Conn_01x03, J17 Conn_01x03, J18 Conn_01x03, J19 Conn_01x03, J2 Conn_01x03, J20 Conn_01x03, J21 Conn_01x03, J22 Conn_01x03, J23 Conn_01x03, J24 Conn_01x03, J25 Conn_01x03, J26 Conn_01x03, J27 Conn_01x03, J28 Conn_01x03, J29 Conn_01x03, J3 Conn_01x03, J30 Conn_02x01, J31 Conn_01x03, J32 Conn_01x04, J33 Conn_01x03, J35 Conn_02x05_Odd_Even, J36 Conn_01x03, J37 Conn_02x20_Odd_Even, J38 Conn_01x03, J39 Conn_01x03, J4 Conn_01x03, J40 Conn_01x03, J41 Conn_01x03, J42 Conn_01x03, J43 Conn_01x03, J5 Conn_01x03, J6 Conn_01x03, J7 Conn_01x03, J8 Conn_01x03, J9 Conn_01x03, Q2 ULN2803ADWR, Q3 ULN2803ADWR, SW1 SW_DIP_x08, U1 ST3232ECDR‎, U2 LPC546xxJyyyBD208, U3 SN65HVD232, Y1 12MHz

Commit message: Rev 1.1 first manufacturable draft.
Parts:
- C32, C33: value 27pF -> 12pF; Digi-Key_PN (none) -> 445-6854-1-ND
- J10, J11, J12, J13, J14, J15, J16, J17, J18, J19, J2, J20, J21, J22, J23, J24, J25, J26, J27, J28, J29, J3, J31, J33, J36, J38, J39, J4, J40, J41, J42, J43, J5, J6, J7, J8, J9: Digi-Key_PN (none) -> 2057-PH1-03-UA-ND
- J30: Digi-Key_PN (none) -> 2057-PH1-02-UA-ND
- J32: Digi-Key_PN (none) -> 2057-PH1-04-UA-ND
- J37: Digi-Key_PN (none) -> PH2-20-UA
- R10: Digi-Key_PN (none) -> 311-120HRCT-ND
- R11, R12: Digi-Key_PN 311-3.30KHRCT-ND -> 311-2.20KHRCT-ND
- R20, R22, R24, R26, R28, R30, R32, R34: Digi-Key_PN 311-3.30KHRCT-ND -> 311-33.0KHRCT-ND
- R21, R23, R25, R27, R29, R31, R33, R35: Digi-Key_PN 311-3.30KHRCT-ND -> 311-27.0KHRCT-ND
- R36: Digi-Key_PN (none) -> 311-33.0KHRCT-ND
- R37: Digi-Key_PN (none) -> 311-3.30KHRCT-ND
- R38: Digi-Key_PN 311-3.30KHRCT-ND -> 311-12.1KHRCT-ND
- RN1: Digi-Key_PN (none) -> 4611X-101-331LF
- SW1: Digi-Key_PN (none) -> CT2108MS-ND
- U1: value ST3232ECDR‎ -> ST3232ECDR; Digi-Key_PN 497-6537-1-ND‎ -> 497-6537-1-ND; MPN ST3232ECDR‎ -> ST3232ECDR
- U2: value LPC546xxJyyyBD208 -> LPC54606J512BD208; Digi-Key_PN (none) -> 568-13367-ND
- U3: Digi-Key_PN 296-26344-1-ND‎ -> 296-26344-1-ND
- Y1: Digi-Key_PN 644-1034-1-nd -> 644-1034-1-ND

Commit message: Correct CPU AVSSC pin.
Other:
- note added: "SWAP order of LEDS here and on the PIO pins!"
Changed lines of the file:
@@
 	7900 4800 8650 4800
 Connection ~ 8650 4700
-Wire Wire Line
-	8650 4300 8650 4150
-Wire Wire Line
-	7900 4300 8650 4300
-Wire Wire Line
-	8650 4300 8650 4600
-Connection ~ 8650 4300
 NoConn ~ 7900 4500
 Wire Wire Line
@@
 AR Path="/6668148C" Ref="R38"  Part="1"
 AR Path="/5CF9559A/6668148C" Ref="R?"  Part="1"
-F 0 "R38" V 8050 4400 50  0000 C CNN
+F 0 "R38" V 8250 4400 50  0000 C CNN
 F 1 "12K1" V 8150 4400 50  0000 C CNN
 F 2 "Resistor_SMD:R_0603_1608Metric_Pad1.05x0.95mm_HandSolder" V 8080 4400 50  0001 C CNN
@@
 	1    0    0    -1
 $EndComp
+Wire Wire Line
+	8650 4150 8650 4600
+Wire Wire Line
+	7900 4300 8550 4300
+Wire Wire Line
+	8550 4300 8550 4400
+Connection ~ 8550 4400
+Text Notes 2750 6550 0    50   Italic 10
+SWAP order of LEDS here and on the PIO pins!
 $EndSCHEMATC

Commit message: Fixed power on VSSC pin, add filter caps, power & reset jumpers, SWD.
Parts:
- removed RN1: 330, Resistor_THT:R_Array_SIP11, symbol Device:R_Network10
- added J44, J45: Conn_01x02, Connector_PinHeader_2.54mm:PinHeader_1x02_P2.54mm_Vertical, symbol Connector_Generic:Conn_01x02
- added R39, R40, R41, R42, R43, R44, R45, R46, R47, R48: 330, Resistor_SMD:R_0603_1608Metric_Pad1.05x0.95mm_HandSolder, symbol Device:R
- R20, R22, R24, R26, R28, R30, R32, R34: value 33K -> 5K; Digi-Key_PN 311-33.0KHRCT-ND -> (none)
- R21, R23, R25, R27, R29, R31, R33, R35: value 27K -> 5K; Digi-Key_PN 311-27.0KHRCT-ND -> (none)
Connections:
- net labels added: SWCLK, SWDIO
- wire segments 595 -> 620
- no-connect marks 125 -> 120
Other:
- note added: "AI0"
- note added: "AI1"
- note added: "AI2"
- note added: "AI3"
- note added: "AI4"
- note added: "AI5"
- note added: "AI6"
- note added: "AI7"
- note removed: "SWAP order of LEDS here and on the PIO pins!"
- moved on the sheet: J2, J3, J37, J4, J40, J41, J42, J43, J5, R20, R21, R22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
