File: POWER.sch (KiCad schematic (older format))
At the start: 44 parts, among them J34 TBL001-500-02GY-2GY, U4 FAN8303, U5 FAN8303, U6 NCP1117ST50T3G, U7 FAN8303

Commit message: Rev 1.1 first manufacturable draft.
Parts:
- C15, C17, C25, C27, C28: Digi-Key_PN (none) -> 1276-1075-1-ND
- C16, C18, C21, C22, C26, C30: Digi-Key_PN (none) -> 1292-1386-1-ND
- C23: value 146pF -> 390pF; Digi-Key_PN (none) -> 1276-2049-1-ND
- C24: value 146pF -> 560pF; Digi-Key_PN (none) -> 1276-1278-1-ND
- C31: value 146pF -> 820pF; Digi-Key_PN (none) -> 1276-2117-1-ND
- J34: Digi-Key_PN (none) -> 102-6360-ND
- L1, L2: value 15uH -> 22uH; footprint Inductor_SMD:L_Taiyo-Yuden_NR-60xx_HandSoldering -> Inductor_SMD:L_Taiyo-Yuden_NR-80xx_HandSoldering; Digi-Key_PN 587-2633-1-ND‎ -> 587-2002-1-ND; MPN (none) -> NR8040T220M
- L3: Digi-Key_PN 587-2633-1-ND‎ -> 587-2633-1-ND
- R13: value X -> 3K; Digi-Key_PN X -> 311-3.00KHRCT-ND
- R14: value X -> 2K45; Digi-Key_PN X -> 311-2.43KHRCT-ND
- R15: value 145K -> 56K; Digi-Key_PN 311-3.30KHRCT-ND -> CR0603-JW-563ELFCT-ND
- R16: value 145K -> 43K; Digi-Key_PN 311-3.30KHRCT-ND -> 311-43.0KHRCT-ND
- R17, R3, R4: value X -> 18K; Digi-Key_PN X -> 311-18.0KHRCT-ND
- R18: value X -> 4K; Digi-Key_PN X -> 311-4.02KHRCT-ND
- R19: value 145K -> 27K; Digi-Key_PN 311-3.30KHRCT-ND -> 311-27.0KHRCT-ND
- U4, U5, U7: Digi-Key_PN (none) -> FAN8303MXCT-ND

Commit message: Fixed power on VSSC pin, add filter caps, power & reset jumpers, SWD.
Parts:
- added C38: 22uF, Capacitor_SMD:C_0805_2012Metric_Pad1.15x1.40mm_HandSolder, symbol Device:C
- added C39, C40, C41: 10uF, Capacitor_SMD:C_1206_3216Metric_Pad1.42x1.75mm_HandSolder, symbol Device:C
- C19, C20, C34, C35: Digi-Key_PN 445-3478-1-ND -> 1276-6780-1-ND
- C29: footprint Capacitor_SMD:C_1210_3225Metric_Pad1.42x2.65mm_HandSolder -> Capacitor_SMD:C_0805_2012Metric_Pad1.15x1.40mm_HandSolder; Digi-Key_PN 445-3478-1-ND -> 1276-6780-1-ND
- R13: value 3K -> 2K; Digi-Key_PN 311-3.00KHRCT-ND -> (none)
Connections:
- net +3V3: now also C38.1
- net +BATT: now also C39.1, C40.1, C41.1
- net GND: now also C38.2, C39.2, C40.2, C41.2
Changed lines of the file:
@@
 Sheet 2 2
 Title "ORIO Power"
-Date "2019-10-07"
-Rev "1.1"
+Date "2019-11-02"
+Rev "1.2"
 Comp ""
 Comment1 ""
@@
 F 0 "C29" H 12415 6596 50  0000 L CNN
 F 1 "22uF" H 12415 6505 50  0000 L CNN
-F 2 "Capacitor_SMD:C_1210_3225Metric_Pad1.42x2.65mm_HandSolder" H 12338 6400 50  0001 C CNN
+F 2 "Capacitor_SMD:C_0805_2012Metric_Pad1.15x1.40mm_HandSolder" H 12338 6400 50  0001 C CNN
 F 3 "~" H 12300 6550 50  0001 C CNN
-F 4 "445-3478-1-ND" H 12700 6300 50  0001 C CNN "Digi-Key_PN"
+F 4 "1276-6780-1-ND" H 12700 6300 50  0001 C CNN "Digi-Key_PN"
 	1    12300 6550
 	1    0    0    -1
@@
 F 2 "Capacitor_SMD:C_1210_3225Metric_Pad1.42x2.65mm_HandSolder" H 12138 3750 50  0001 C CNN
 F 3 "~" H 12100 3900 50  0001 C CNN
-F 4 "445-3478-1-ND" H 12500 3650 50  0001 C CNN "Digi-Key_PN"
+F 4 "1276-6780-1-ND" H 12500 3650 50  0001 C CNN "Digi-Key_PN"
 	1    12100 3900
 	1    0    0    -1
@@
 AR Path="/5DFE66B1/5E0E83D9" Ref="R13"  Part="1"
 F 0 "R13" V 6200 3950 50  0000 C CNN
-F 1 "3K" V 6300 3950 50  0000 C CNN
+F 1 "2K" V 6300 3950 50  0000 C CNN
 F 2 "Resistor_SMD:R_0603_1608Metric_Pad1.05x0.95mm_HandSolder" V 6230 3950 50  0001 C CNN
 F 3 "~" H 6300 3950 50  0001 C CNN
-F 4 "311-3.00KHRCT-ND" H 6300 3950 50  0001 C CNN "Digi-Key_PN"
+F 4 "" H 6300 3950 50  0001 C CNN "Digi-Key_PN"
 	1    6300 3950
 	-1   0    0    1
@@
 F 2 "Capacitor_SMD:C_1210_3225Metric_Pad1.42x2.65mm_HandSolder" H 6688 3600 50  0001 C CNN
 F 3 "~" H 6650 3750 50  0001 C CNN
-F 4 "445-3478-1-ND" H 7050 3500 50  0001 C CNN "Digi-Key_PN"
+F 4 "1276-6780-1-ND" H 7050 3500 50  0001 C CNN "Digi-Key_PN"
 	1    6650 3750
 	1    0    0    -1
@@
 L power:+BATT #PWR0120
 U 1 1 600D6FA6
-P 4550 7850
-F 0 "#PWR0120" H 4550 7700 50  0001 C CNN
-F 1 "+BATT" H 4565 8023 50  0000 C CNN
-F 2 "" H 4550 7850 50  0001 C CNN
-F 3 "" H 4550 7850 50  0001 C CNN
-	1    4550 7850
+P 5350 7850
+F 0 "#PWR0120" H 5350 7700 50  0001 C CNN
+F 1 "+BATT" H 5365 8023 50  0000 C CNN
+F 2 "" H 5350 7850 50  0001 C CNN
+F 3 "" H 5350 7850 50  0001 C CNN
+	1    5350 7850
 	1    0    0    -1
 $EndComp
@@
 Connection ~ 12450 6200
 Wire Wire Line
-	12450 6200 12800 6200
+	12450 6200 12750 6200
 Text Notes 2600 8700 0    50   ~ 0
 12V Battery
@@
 F 2 "Capacitor_SMD:C_1210_3225Metric_Pad1.42x2.65mm_HandSolder" H 12638 3750 50  0001 C CNN
 F 3 "~" H 12600 3900 50  0001 C CNN
-F 4 "445-3478-1-ND" H 13000 3650 50  0001 C CNN "Digi-Key_PN"
+F 4 "1276-6780-1-ND" H 13000 3650 50  0001 C CNN "Digi-Key_PN"
 	1    12600 3900
 	1    0    0    -1
@@
 F 2 "Capacitor_SMD:C_1210_3225Metric_Pad1.42x2.65mm_HandSolder" H 13088 3750 50  0001 C CNN
 F 3 "~" H 13050 3900 50  0001 C CNN
-F 4 "445-3478-1-ND" H 13450 3650 50  0001 C CNN "Digi-Key_PN"
+F 4 "1276-6780-1-ND" H 13450 3650 50  0001 C CNN "Digi-Key_PN"
 	1    13050 3900
 	1    0    0    -1
@@
 Connection ~ 3950 7850
 Wire Wire Line
-	3950 7850 4550 7850
+	3950 7850 4100 7850
 $Comp
 L JWlib:NCP1117ST50T3G U6
@@
 	1    0    0    -1
 $EndComp
+$Comp
+L Device:C C?
+U 1 1 5E30C54F
+P 12750 6550
+AR Path="/5BBE5CCD/5E30C54F" Ref="C?"  Part="1"
+AR Path="/5E30C54F" Ref="C?"  Part="1"
+AR Path="/5CF9559A/5E30C54F" Ref="C?"  Part="1"
+AR Path="/5DFE66B1/5E30C54F" Ref="C38"  Part="1"
+F 0 "C38" H 12865 6596 50  0000 L CNN
+F 1 "22uF" H 12865 6505 50  0000 L CNN
+F 2 "Capacitor_SMD:C_0805_2012Metric_Pad1.15x1.40mm_HandSolder" H 12788 6400 50  0001 C CNN
+F 3 "~" H 12750 6550 50  0001 C CNN
+F 4 "1276-6780-1-ND" H 13150 6300 50  0001 C CNN "Digi-Key_PN"
+	1    12750 6550
+	1    0    0    -1
+$EndComp
+Wire Wire Line
+	12750 6400 12750 6200
+Connection ~ 12750 6200
+Wire Wire Line
+	12750 6200 12800 6200
+Wire Wire Line
+	12750 6700 12750 7500
+Wire Wire Line
+	12750 7500 12300 7500
+Connection ~ 12300 7500
+$Comp
+L Device:C C?
+U 1 1 5E31A8B4
+P 4100 8000
+AR Path="/5BBE5CCD/5E31A8B4" Ref="C?"  Part="1"
+AR Path="/5E31A8B4" Ref="C?"  Part="1"
+AR Path="/5CF9559A/5E31A8B4" Ref="C?"  Part="1"
+AR Path="/5DFE66B1/5E31A8B4" Ref="C39"  Part="1"
+F 0 "C39" H 4215 8046 50  0000 L CNN
+F 1 "10uF" H 4215 7955 50  0000 L CNN
+F 2 "Capacitor_SMD:C_1206_3216Metric_Pad1.42x1.75mm_HandSolder" H 4138 7850 50  0001 C CNN
+F 3 "~" H 4100 8000 50  0001 C CNN
+F 4 " 1276-1075-1-ND " H 4500 7750 50  0001 C CNN "Digi-Key_PN"
+	1    4100 8000
+	1    0    0    -1
+$EndComp
+$Comp
+L Device:C C?
+U 1 1 5E321E39
+P 4550 8000
+AR Path="/5BBE5CCD/5E321E39" Ref="C?"  Part="1"
+AR Path="/5E321E39" Ref="C?"  Part="1"
+AR Path="/5CF9559A/5E321E39" Ref="C?"  Part="1"
+AR Path="/5DFE66B1/5E321E39" Ref="C40"  Part="1"
+F 0 "C40" H 4665 8046 50  0000 L CNN
+F 1 "10uF" H 4665 7955 50  0000 L CNN
+F 2 "Capacitor_SMD:C_1206_3216Metric_Pad1.42x1.75mm_HandSolder" H 4588 7850 50  0001 C CNN
+F 3 "~" H 4550 8000 50  0001 C CNN
+F 4 " 1276-1075-1-ND " H 4950 7750 50  0001 C CNN "Digi-Key_PN"
+	1    4550 8000
+	1    0    0    -1
+$EndComp
+$Comp
+L Device:C C?
+U 1 1 5E3222FC
+P 5000 8000
+AR Path="/5BBE5CCD/5E3222FC" Ref="C?"  Part="1"
+AR Path="/5E3222FC" Ref="C?"  Part="1"
+AR Path="/5CF9559A/5E3222FC" Ref="C?"  Part="1"
+AR Path="/5DFE66B1/5E3222FC" Ref="C41"  Part="1"
+F 0 "C41" H 5115 8046 50  0000 L CNN
+F 1 "10uF" H 5115 7955 50  0000 L CNN
+F 2 "Capacitor_SMD:C_1206_3216Metric_Pad1.42x1.75mm_HandSolder" H 5038 7850 50  0001 C CNN
+F 3 "~" H 5000 8000 50  0001 C CNN
+F 4 " 1276-1075-1-ND " H 5400 7750 50  0001 C CNN "Digi-Key_PN"
+	1    5000 8000
+	1    0    0    -1
+$EndComp
+Connection ~ 5000 7850
+Wire Wire Line
+	5000 7850 5350 7850
+Wire Wire Line
+	4100 7850 4550 7850
+Connection ~ 4100 7850
+Connection ~ 4550 7850
+Wire Wire Line
+	4550 7850 5000 7850
+Wire Wire Line
+	4100 8150 4350 8150
+Connection ~ 4550 8150
+Wire Wire Line
+	4550 8150 5000 8150
+$Comp
+L power:GND #PWR?
+U 1 1 5E3302F8
+P 4350 8150
+AR Path="/5E3302F8" Ref="#PWR?"  Part="1"
+AR Path="/5DFE66B1/5E3302F8" Ref="#PWR035"  Part="1"
+F 0 "#PWR035" H 4350 7900 50  0001 C CNN
+F 1 "GND" H 4355 7977 50  0000 C CNN
+F 2 "" H 4350 8150 50  0001 C CNN
+F 3 "" H 4350 8150 50  0001 C CNN
+	1    4350 8150
+	1    0    0    -1
+$EndComp
+Connection ~ 4350 8150
+Wire Wire Line
+	4350 8150 4550 8150
 $EndSCHEMATC
